File: PCB/Santas Microfactory - Backplane/Santas Microfactory - Backplane.kicad_sch (KiCad schematic)
At the start: 0 parts

Commit message: More work
Parts:
- added CN1, CN2, CN3, CN4, CN5, CN6, CN7: 2EG08217-D2D-DF, imported_components:CONN-TH_2EG08217-D2D-DF, symbol imported_components:2EG08217-D2D-DF
- added H1, H2, H3, H4, H5, H6: MountingHole, MountingHole:MountingHole_3.2mm_M3_Pad_Via, symbol Mechanical:MountingHole
Connections:
- new net A1: CN1.1 (A1), CN2.1 (A1), CN3.1 (A1), CN4.1 (A1), CN5.1 (A1), CN6.1 (A1), CN7.1 (A1)
- new net A10: CN1.10 (A10), CN2.10 (A10), CN3.10 (A10), CN4.10 (A10), CN5.10 (A10), CN6.10 (A10), CN7.10 (A10)
- new net A11: CN1.11 (A11), CN2.11 (A11), CN3.11 (A11), CN4.11 (A11), CN5.11 (A11), CN6.11 (A11), CN7.11 (A11)
- new net A12: CN1.12 (A12), CN2.12 (A12), CN3.12 (A12), CN4.12 (A12), CN5.12 (A12), CN6.12 (A12), CN7.12 (A12)
- new net A13: CN1.13 (A13), CN2.13 (A13), CN3.13 (A13), CN4.13 (A13), CN5.13 (A13), CN6.13 (A13), CN7.13 (A13)
- new net A14: CN1.14 (A14), CN2.14 (A14), CN3.14 (A14), CN4.14 (A14), CN5.14 (A14), CN6.14 (A14), CN7.14 (A14)
- new net A15: CN1.15 (A15), CN2.15 (A15), CN3.15 (A15), CN4.15 (A15), CN5.15 (A15), CN6.15 (A15), CN7.15 (A15)
- new net A16: CN1.16 (A16), CN2.16 (A16), CN3.16 (A16), CN4.16 (A16), CN5.16 (A16), CN6.16 (A16), CN7.16 (A16)
- new net A17: CN1.17 (A17), CN2.17 (A17), CN3.17 (A17), CN4.17 (A17), CN5.17 (A17), CN6.17 (A17), CN7.17 (A17)
- new net A18: CN1.18 (A18), CN2.18 (A18), CN3.18 (A18), CN4.18 (A18), CN5.18 (A18), CN6.18 (A18), CN7.18 (A18)
- new net A19: CN1.19 (A19), CN2.19 (A19), CN3.19 (A19), CN4.19 (A19), CN5.19 (A19), CN6.19 (A19), CN7.19 (A19)
- new net A2: CN1.2 (A2), CN2.2 (A2), CN3.2 (A2), CN4.2 (A2), CN5.2 (A2), CN6.2 (A2), CN7.2 (A2)
- new net A20: CN1.20 (A20), CN2.20 (A20), CN3.20 (A20), CN4.20 (A20), CN5.20 (A20), CN6.20 (A20), CN7.20 (A20)
- new net A21: CN1.21 (A21), CN2.21 (A21), CN3.21 (A21), CN4.21 (A21), CN5.21 (A21), CN6.21 (A21), CN7.21 (A21)
- new net A22: CN1.22 (A22), CN2.22 (A22), CN3.22 (A22), CN4.22 (A22), CN5.22 (A22), CN6.22 (A22), CN7.22 (A22)
- new net A23: CN1.23 (A23), CN2.23 (A23), CN3.23 (A23), CN4.23 (A23), CN5.23 (A23), CN6.23 (A23), CN7.23 (A23)
- new net A24: CN1.24 (A24), CN2.24 (A24), CN3.24 (A24), CN4.24 (A24), CN5.24 (A24), CN6.24 (A24), CN7.24 (A24)
- new net A25: CN1.25 (A25), CN2.25 (A25), CN3.25 (A25), CN4.25 (A25), CN5.25 (A25), CN6.25 (A25), CN7.25 (A25)
- new net A26: CN1.26 (A26), CN2.26 (A26), CN3.26 (A26), CN4.26 (A26), CN5.26 (A26), CN6.26 (A26), CN7.26 (A26)
- new net A27: CN1.27 (A27), CN2.27 (A27), CN3.27 (A27), CN4.27 (A27), CN5.27 (A27), CN6.27 (A27), CN7.27 (A27)
- new net A28: CN1.28 (A28), CN2.28 (A28), CN3.28 (A28), CN4.28 (A28), CN5.28 (A28), CN6.28 (A28), CN7.28 (A28)
- new net A29: CN1.29 (A29), CN2.29 (A29), CN3.29 (A29), CN4.29 (A29), CN5.29 (A29), CN6.29 (A29), CN7.29 (A29)
- new net A3: CN1.3 (A3), CN2.3 (A3), CN3.3 (A3), CN4.3 (A3), CN5.3 (A3), CN6.3 (A3), CN7.3 (A3)
- new net A30: CN1.30 (A30), CN2.30 (A30), CN3.30 (A30), CN4.30 (A30), CN5.30 (A30), CN6.30 (A30), CN7.30 (A30)
- new net A31: CN1.31 (A31), CN2.31 (A31), CN3.31 (A31), CN4.31 (A31), CN5.31 (A31), CN6.31 (A31), CN7.31 (A31)
- new net A32: CN1.32 (A32), CN2.32 (A32), CN3.32 (A32), CN4.32 (A32), CN5.32 (A32), CN6.32 (A32), CN7.32 (A32)
- new net A33: CN1.33 (A33), CN2.33 (A33), CN3.33 (A33), CN4.33 (A33), CN5.33 (A33), CN6.33 (A33), CN7.33 (A33)
- new net A34: CN1.34 (A34), CN2.34 (A34), CN3.34 (A34), CN4.34 (A34), CN5.34 (A34), CN6.34 (A34), CN7.34 (A34)
- new net A35: CN1.35 (A35), CN2.35 (A35), CN3.35 (A35), CN4.35 (A35), CN5.35 (A35), CN6.35 (A35), CN7.35 (A35)
- new net A36: CN1.36 (A36), CN2.36 (A36), CN3.36 (A36), CN4.36 (A36), CN5.36 (A36), CN6.36 (A36), CN7.36 (A36)
- new net A37: CN1.37 (A37), CN2.37 (A37), CN3.37 (A37), CN4.37 (A37), CN5.37 (A37), CN6.37 (A37), CN7.37 (A37)
- new net A38: CN1.38 (A38), CN2.38 (A38), CN3.38 (A38), CN4.38 (A38), CN5.38 (A38), CN6.38 (A38), CN7.38 (A38)
- new net A39: CN1.39 (A39), CN2.39 (A39), CN3.39 (A39), CN4.39 (A39), CN5.39 (A39), CN6.39 (A39), CN7.39 (A39)
- new net A4: CN1.4 (A4), CN2.4 (A4), CN3.4 (A4), CN4.4 (A4), CN5.4 (A4), CN6.4 (A4), CN7.4 (A4)
- new net A40: CN1.40 (A40), CN2.40 (A40), CN3.40 (A40), CN4.40 (A40), CN5.40 (A40), CN6.40 (A40), CN7.40 (A40)
- new net A41: CN1.41 (A41), CN2.41 (A41), CN3.41 (A41), CN4.41 (A41), CN5.41 (A41), CN6.41 (A41), CN7.41 (A41)
- new net A42: CN1.42 (A42), CN2.42 (A42), CN3.42 (A42), CN4.42 (A42), CN5.42 (A42), CN6.42 (A42), CN7.42 (A42)
- new net A43: CN1.43 (A43), CN2.43 (A43), CN3.43 (A43), CN4.43 (A43), CN5.43 (A43), CN6.43 (A43), CN7.43 (A43)
- new net A44: CN1.44 (A44), CN2.44 (A44), CN3.44 (A44), CN4.44 (A44), CN5.44 (A44), CN6.44 (A44), CN7.44 (A44)
- new net A45: CN1.45 (A45), CN2.45 (A45), CN3.45 (A45), CN4.45 (A45), CN5.45 (A45), CN6.45 (A45), CN7.45 (A45)
- new net A46: CN1.46 (A46), CN2.46 (A46), CN3.46 (A46), CN4.46 (A46), CN5.46 (A46), CN6.46 (A46), CN7.46 (A46)
- new net A47: CN1.47 (A47), CN2.47 (A47), CN3.47 (A47), CN4.47 (A47), CN5.47 (A47), CN6.47 (A47), CN7.47 (A47)
- new net A48: CN1.48 (A48), CN2.48 (A48), CN3.48 (A48), CN4.48 (A48), CN5.48 (A48), CN6.48 (A48), CN7.48 (A48)
- new net A49: CN1.49 (A49), CN2.49 (A49), CN3.49 (A49), CN4.49 (A49), CN5.49 (A49), CN6.49 (A49), CN7.49 (A49)
- new net A5: CN1.5 (A5), CN2.5 (A5), CN3.5 (A5), CN4.5 (A5), CN5.5 (A5), CN6.5 (A5), CN7.5 (A5)
- new net A50: CN1.50 (A50), CN2.50 (A50), CN3.50 (A50), CN4.50 (A50), CN5.50 (A50), CN6.50 (A50), CN7.50 (A50)
- new net A51: CN1.51 (A51), CN2.51 (A51), CN3.51 (A51), CN4.51 (A51), CN5.51 (A51), CN6.51 (A51), CN7.51 (A51)
- new net A52: CN1.52 (A52), CN2.52 (A52), CN3.52 (A52), CN4.52 (A52), CN5.52 (A52), CN6.52 (A52), CN7.52 (A52)
- new net A53: CN1.53 (A53), CN2.53 (A53), CN3.53 (A53), CN4.53 (A53), CN5.53 (A53), CN6.53 (A53), CN7.53 (A53)
- new net A54: CN1.54 (A54), CN2.54 (A54), CN3.54 (A54), CN4.54 (A54), CN5.54 (A54), CN6.54 (A54), CN7.54 (A54)
- new net A55: CN1.55 (A55), CN2.55 (A55), CN3.55 (A55), CN4.55 (A55), CN5.55 (A55), CN6.55 (A55), CN7.55 (A55)
- new net A56: CN1.56 (A56), CN2.56 (A56), CN3.56 (A56), CN4.56 (A56), CN5.56 (A56), CN6.56 (A56), CN7.56 (A56)
- new net A57: CN1.57 (A57), CN2.57 (A57), CN3.57 (A57), CN4.57 (A57), CN5.57 (A57), CN6.57 (A57), CN7.57 (A57)
- new net A58: CN1.58 (A58), CN2.58 (A58), CN3.58 (A58), CN4.58 (A58), CN5.58 (A58), CN6.58 (A58), CN7.58 (A58)
- new net A59: CN1.59 (A59), CN2.59 (A59), CN3.59 (A59), CN4.59 (A59), CN5.59 (A59), CN6.59 (A59), CN7.59 (A59)
- new net A6: CN1.6 (A6), CN2.6 (A6), CN3.6 (A6), CN4.6 (A6), CN5.6 (A6), CN6.6 (A6), CN7.6 (A6)
- new net A60: CN1.60 (A60), CN2.60 (A60), CN3.60 (A60), CN4.60 (A60), CN5.60 (A60), CN6.60 (A60), CN7.60 (A60)
- new net A61: CN1.61 (A61), CN2.61 (A61), CN3.61 (A61), CN4.61 (A61), CN5.61 (A61), CN6.61 (A61), CN7.61 (A61)
- new net A62: CN1.62 (A62), CN2.62 (A62), CN3.62 (A62), CN4.62 (A62), CN5.62 (A62), CN6.62 (A62), CN7.62 (A62)
- new net A63: CN1.63 (A63), CN2.63 (A63), CN3.63 (A63), CN4.63 (A63), CN5.63 (A63), CN6.63 (A63), CN7.63 (A63)
- new net A64: CN1.64 (A64), CN2.64 (A64), CN3.64 (A64), CN4.64 (A64), CN5.64 (A64), CN6.64 (A64), CN7.64 (A64)
- new net A65: CN1.65 (A65), CN2.65 (A65), CN3.65 (A65), CN4.65 (A65), CN5.65 (A65), CN6.65 (A65), CN7.65 (A65)
- new net A66: CN1.66 (A66), CN2.66 (A66), CN3.66 (A66), CN4.66 (A66), CN5.66 (A66), CN6.66 (A66), CN7.66 (A66)
- new net A67: CN1.67 (A67), CN2.67 (A67), CN3.67 (A67), CN4.67 (A67), CN5.67 (A67), CN6.67 (A67), CN7.67 (A67)
- new net A68: CN1.68 (A68), CN2.68 (A68), CN3.68 (A68), CN4.68 (A68), CN5.68 (A68), CN6.68 (A68), CN7.68 (A68)
- new net A69: CN1.69 (A69), CN2.69 (A69), CN3.69 (A69), CN4.69 (A69), CN5.69 (A69), CN6.69 (A69), CN7.69 (A69)
- new net A7: CN1.7 (A7), CN2.7 (A7), CN3.7 (A7), CN4.7 (A7), CN5.7 (A7), CN6.7 (A7), CN7.7 (A7)
- new net A70: CN1.70 (A70), CN2.70 (A70), CN3.70 (A70), CN4.70 (A70), CN5.70 (A70), CN6.70 (A70), CN7.70 (A70)
- new net A71: CN1.71 (A71), CN2.71 (A71), CN3.71 (A71), CN4.71 (A71), CN5.71 (A71), CN6.71 (A71), CN7.71 (A71)
- new net A72: CN1.72 (A72), CN2.72 (A72), CN3.72 (A72), CN4.72 (A72), CN5.72 (A72), CN6.72 (A72), CN7.72 (A72)
- new net A73: CN1.73 (A73), CN2.73 (A73), CN3.73 (A73), CN4.73 (A73), CN5.73 (A73), CN6.73 (A73), CN7.73 (A73)
- new net A74: CN1.74 (A74), CN2.74 (A74), CN3.74 (A74), CN4.74 (A74), CN5.74 (A74), CN6.74 (A74), CN7.74 (A74)
- new net A75: CN1.75 (A75), CN2.75 (A75), CN3.75 (A75), CN4.75 (A75), CN5.75 (A75), CN6.75 (A75), CN7.75 (A75)
- new net A76: CN1.76 (A76), CN2.76 (A76), CN3.76 (A76), CN4.76 (A76), CN5.76 (A76), CN6.76 (A76), CN7.76 (A76)
- new net A77: CN1.77 (A77), CN2.77 (A77), CN3.77 (A77), CN4.77 (A77), CN5.77 (A77), CN6.77 (A77), CN7.77 (A77)
- new net A78: CN1.78 (A78), CN2.78 (A78), CN3.78 (A78), CN4.78 (A78), CN5.78 (A78), CN6.78 (A78), CN7.78 (A78)
- new net A79: CN1.79 (A79), CN2.79 (A79), CN3.79 (A79), CN4.79 (A79), CN5.79 (A79), CN6.79 (A79), CN7.79 (A79)
- new net A8: CN1.8 (A8), CN2.8 (A8), CN3.8 (A8), CN4.8 (A8), CN5.8 (A8), CN6.8 (A8), CN7.8 (A8)
- new net A80: CN1.80 (A80), CN2.80 (A80), CN3.80 (A80), CN4.80 (A80), CN5.80 (A80), CN6.80 (A80), CN7.80 (A80)
- new net A81: CN1.81 (A81), CN2.81 (A81), CN3.81 (A81), CN4.81 (A81), CN5.81 (A81), CN6.81 (A81), CN7.81 (A81)
- new net A82: CN1.82 (A82), CN2.82 (A82), CN3.82 (A82), CN4.82 (A82), CN5.82 (A82), CN6.82 (A82), CN7.82 (A82)
- new net A9: CN1.9 (A9), CN2.9 (A9), CN3.9 (A9), CN4.9 (A9), CN5.9 (A9), CN6.9 (A9), CN7.9 (A9)
- new net B1: CN1.83 (B1), CN2.83 (B1), CN3.83 (B1), CN4.83 (B1), CN5.83 (B1), CN6.83 (B1), CN7.83 (B1)
- new net B10: CN1.92 (B10), CN2.92 (B10), CN3.92 (B10), CN4.92 (B10), CN5.92 (B10), CN6.92 (B10), CN7.92 (B10)
- new net B11: CN1.93 (B11), CN2.93 (B11), CN3.93 (B11), CN4.93 (B11), CN5.93 (B11), CN6.93 (B11), CN7.93 (B11)
- new net B12: CN1.94 (B12), CN2.94 (B12), CN3.94 (B12), CN4.94 (B12), CN5.94 (B12), CN6.94 (B12), CN7.94 (B12)
- new net B13: CN1.95 (B13), CN2.95 (B13), CN3.95 (B13), CN4.95 (B13), CN5.95 (B13), CN6.95 (B13), CN7.95 (B13)
- new net B14: CN1.96 (B14), CN2.96 (B14), CN3.96 (B14), CN4.96 (B14), CN5.96 (B14), CN6.96 (B14), CN7.96 (B14)
- new net B15: CN1.97 (B15), CN2.97 (B15), CN3.97 (B15), CN4.97 (B15), CN5.97 (B15), CN6.97 (B15), CN7.97 (B15)
- new net B16: CN1.98 (B16), CN2.98 (B16), CN3.98 (B16), CN4.98 (B16), CN5.98 (B16), CN6.98 (B16), CN7.98 (B16)
- new net B17: CN1.99 (B17), CN2.99 (B17), CN3.99 (B17), CN4.99 (B17), CN5.99 (B17), CN6.99 (B17), CN7.99 (B17)
- new net B18: CN1.100 (B18), CN2.100 (B18), CN3.100 (B18), CN4.100 (B18), CN5.100 (B18), CN6.100 (B18), CN7.100 (B18)
- new net B19: CN1.101 (B19), CN2.101 (B19), CN3.101 (B19), CN4.101 (B19), CN5.101 (B19), CN6.101 (B19), CN7.101 (B19)
- new net B2: CN1.84 (B2), CN2.84 (B2), CN3.84 (B2), CN4.84 (B2), CN5.84 (B2), CN6.84 (B2), CN7.84 (B2)
- new net B20: CN1.102 (B20), CN2.102 (B20), CN3.102 (B20), CN4.102 (B20), CN5.102 (B20), CN6.102 (B20), CN7.102 (B20)
- new net B21: CN1.103 (B21), CN2.103 (B21), CN3.103 (B21), CN4.103 (B21), CN5.103 (B21), CN6.103 (B21), CN7.103 (B21)
- new net B22: CN1.104 (B22), CN2.104 (B22), CN3.104 (B22), CN4.104 (B22), CN5.104 (B22), CN6.104 (B22), CN7.104 (B22)
- new net B23: CN1.105 (B23), CN2.105 (B23), CN3.105 (B23), CN4.105 (B23), CN5.105 (B23), CN6.105 (B23), CN7.105 (B23)
- new net B24: CN1.106 (B24), CN2.106 (B24), CN3.106 (B24), CN4.106 (B24), CN5.106 (B24), CN6.106 (B24), CN7.106 (B24)
- new net B25: CN1.107 (B25), CN2.107 (B25), CN3.107 (B25), CN4.107 (B25), CN5.107 (B25), CN6.107 (B25), CN7.107 (B25)
- new net B26: CN1.108 (B26), CN2.108 (B26), CN3.108 (B26), CN4.108 (B26), CN5.108 (B26), CN6.108 (B26), CN7.108 (B26)
- new net B27: CN1.109 (B27), CN2.109 (B27), CN3.109 (B27), CN4.109 (B27), CN5.109 (B27), CN6.109 (B27), CN7.109 (B27)
- new net B28: CN1.110 (B28), CN2.110 (B28), CN3.110 (B28), CN4.110 (B28), CN5.110 (B28), CN6.110 (B28), CN7.110 (B28)
- new net B29: CN1.111 (B29), CN2.111 (B29), CN3.111 (B29), CN4.111 (B29), CN5.111 (B29), CN6.111 (B29), CN7.111 (B29)
- new net B3: CN1.85 (B3), CN2.85 (B3), CN3.85 (B3), CN4.85 (B3), CN5.85 (B3), CN6.85 (B3), CN7.85 (B3)
- new net B30: CN1.112 (B30), CN2.112 (B30), CN3.112 (B30), CN4.112 (B30), CN5.112 (B30), CN6.112 (B30), CN7.112 (B30)
- new net B31: CN1.113 (B31), CN2.113 (B31), CN3.113 (B31), CN4.113 (B31), CN5.113 (B31), CN6.113 (B31), CN7.113 (B31)
- new net B32: CN1.114 (B32), CN2.114 (B32), CN3.114 (B32), CN4.114 (B32), CN5.114 (B32), CN6.114 (B32), CN7.114 (B32)
- new net B33: CN1.115 (B33), CN2.115 (B33), CN3.115 (B33), CN4.115 (B33), CN5.115 (B33), CN6.115 (B33), CN7.115 (B33)
- new net B34: CN1.116 (B34), CN2.116 (B34), CN3.116 (B34), CN4.116 (B34), CN5.116 (B34), CN6.116 (B34), CN7.116 (B34)
- new net B35: CN1.117 (B35), CN2.117 (B35), CN3.117 (B35), CN4.117 (B35), CN5.117 (B35), CN6.117 (B35), CN7.117 (B35)
- new net B36: CN1.118 (B36), CN2.118 (B36), CN3.118 (B36), CN4.118 (B36), CN5.118 (B36), CN6.118 (B36), CN7.118 (B36)
- new net B37: CN1.119 (B37), CN2.119 (B37), CN3.119 (B37), CN4.119 (B37), CN5.119 (B37), CN6.119 (B37), CN7.119 (B37)
- new net B38: CN1.120 (B38), CN2.120 (B38), CN3.120 (B38), CN4.120 (B38), CN5.120 (B38), CN6.120 (B38), CN7.120 (B38)
- new net B39: CN1.121 (B39), CN2.121 (B39), CN3.121 (B39), CN4.121 (B39), CN5.121 (B39), CN6.121 (B39), CN7.121 (B39)
- new net B4: CN1.86 (B4), CN2.86 (B4), CN3.86 (B4), CN4.86 (B4), CN5.86 (B4), CN6.86 (B4), CN7.86 (B4)
- new net B40: CN1.122 (B40), CN2.122 (B40), CN3.122 (B40), CN4.122 (B40), CN5.122 (B40), CN6.122 (B40), CN7.122 (B40)
- new net B41: CN1.123 (B41), CN2.123 (B41), CN3.123 (B41), CN4.123 (B41), CN5.123 (B41), CN6.123 (B41), CN7.123 (B41)
- new net B42: CN1.124 (B42), CN2.124 (B42), CN3.124 (B42), CN4.124 (B42), CN5.124 (B42), CN6.124 (B42), CN7.124 (B42)
- new net B43: CN1.125 (B43), CN2.125 (B43), CN3.125 (B43), CN4.125 (B43), CN5.125 (B43), CN6.125 (B43), CN7.125 (B43)
- new net B44: CN1.126 (B44), CN2.126 (B44), CN3.126 (B44), CN4.126 (B44), CN5.126 (B44), CN6.126 (B44), CN7.126 (B44)
- new net B45: CN1.127 (B45), CN2.127 (B45), CN3.127 (B45), CN4.127 (B45), CN5.127 (B45), CN6.127 (B45), CN7.127 (B45)
- new net B46: CN1.128 (B46), CN2.128 (B46), CN3.128 (B46), CN4.128 (B46), CN5.128 (B46), CN6.128 (B46), CN7.128 (B46)
- new net B47: CN1.129 (B47), CN2.129 (B47), CN3.129 (B47), CN4.129 (B47), CN5.129 (B47), CN6.129 (B47), CN7.129 (B47)
- new net B48: CN1.130 (B48), CN2.130 (B48), CN3.130 (B48), CN4.130 (B48), CN5.130 (B48), CN6.130 (B48), CN7.130 (B48)
- new net B49: CN1.131 (B49), CN2.131 (B49), CN3.131 (B49), CN4.131 (B49), CN5.131 (B49), CN6.131 (B49), CN7.131 (B49)
- new net B5: CN1.87 (B5), CN2.87 (B5), CN3.87 (B5), CN4.87 (B5), CN5.87 (B5), CN6.87 (B5), CN7.87 (B5)
- new net B50: CN1.132 (B50), CN2.132 (B50), CN3.132 (B50), CN4.132 (B50), CN5.132 (B50), CN6.132 (B50), CN7.132 (B50)
- new net B51: CN1.133 (B51), CN2.133 (B51), CN3.133 (B51), CN4.133 (B51), CN5.133 (B51), CN6.133 (B51), CN7.133 (B51)
- new net B52: CN1.134 (B52), CN2.134 (B52), CN3.134 (B52), CN4.134 (B52), CN5.134 (B52), CN6.134 (B52), CN7.134 (B52)
- new net B53: CN1.135 (B53), CN2.135 (B53), CN3.135 (B53), CN4.135 (B53), CN5.135 (B53), CN6.135 (B53), CN7.135 (B53)
- new net B54: CN1.136 (B54), CN2.136 (B54), CN3.136 (B54), CN4.136 (B54), CN5.136 (B54), CN6.136 (B54), CN7.136 (B54)
- new net B55: CN1.137 (B55), CN2.137 (B55), CN3.137 (B55), CN4.137 (B55), CN5.137 (B55), CN6.137 (B55), CN7.137 (B55)
- new net B56: CN1.138 (B56), CN2.138 (B56), CN3.138 (B56), CN4.138 (B56), CN5.138 (B56), CN6.138 (B56), CN7.138 (B56)
- new net B57: CN1.139 (B57), CN2.139 (B57), CN3.139 (B57), CN4.139 (B57), CN5.139 (B57), CN6.139 (B57), CN7.139 (B57)
- new net B58: CN1.140 (B58), CN2.140 (B58), CN3.140 (B58), CN4.140 (B58), CN5.140 (B58), CN6.140 (B58), CN7.140 (B58)
- new net B59: CN1.141 (B59), CN2.141 (B59), CN3.141 (B59), CN4.141 (B59), CN5.141 (B59), CN6.141 (B59), CN7.141 (B59)
- new net B6: CN1.88 (B6), CN2.88 (B6), CN3.88 (B6), CN4.88 (B6), CN5.88 (B6), CN6.88 (B6), CN7.88 (B6)
- new net B60: CN1.142 (B60), CN2.142 (B60), CN3.142 (B60), CN4.142 (B60), CN5.142 (B60), CN6.142 (B60), CN7.142 (B60)
- new net B61: CN1.143 (B61), CN2.143 (B61), CN3.143 (B61), CN4.143 (B61), CN5.143 (B61), CN6.143 (B61), CN7.143 (B61)
- new net B62: CN1.144 (B62), CN2.144 (B62), CN3.144 (B62), CN4.144 (B62), CN5.144 (B62), CN6.144 (B62), CN7.144 (B62)
- new net B63: CN1.145 (B63), CN2.145 (B63), CN3.145 (B63), CN4.145 (B63), CN5.145 (B63), CN6.145 (B63), CN7.145 (B63)
- new net B64: CN1.146 (B64), CN2.146 (B64), CN3.146 (B64), CN4.146 (B64), CN5.146 (B64), CN6.146 (B64), CN7.146 (B64)
- new net B65: CN1.147 (B65), CN2.147 (B65), CN3.147 (B65), CN4.147 (B65), CN5.147 (B65), CN6.147 (B65), CN7.147 (B65)
- new net B66: CN1.148 (B66), CN2.148 (B66), CN3.148 (B66), CN4.148 (B66), CN5.148 (B66), CN6.148 (B66), CN7.148 (B66)
- new net B67: CN1.149 (B67), CN2.149 (B67), CN3.149 (B67), CN4.149 (B67), CN5.149 (B67), CN6.149 (B67), CN7.149 (B67)
- new net B68: CN1.150 (B68), CN2.150 (B68), CN3.150 (B68), CN4.150 (B68), CN5.150 (B68), CN6.150 (B68), CN7.150 (B68)
- new net B69: CN1.151 (B69), CN2.151 (B69), CN3.151 (B69), CN4.151 (B69), CN5.151 (B69), CN6.151 (B69), CN7.151 (B69)
- new net B7: CN1.89 (B7), CN2.89 (B7), CN3.89 (B7), CN4.89 (B7), CN5.89 (B7), CN6.89 (B7), CN7.89 (B7)
- new net B70: CN1.152 (B70), CN2.152 (B70), CN3.152 (B70), CN4.152 (B70), CN5.152 (B70), CN6.152 (B70), CN7.152 (B70)
- new net B71: CN1.153 (B71), CN2.153 (B71), CN3.153 (B71), CN4.153 (B71), CN5.153 (B71), CN6.153 (B71), CN7.153 (B71)
- new net B72: CN1.154 (B72), CN2.154 (B72), CN3.154 (B72), CN4.154 (B72), CN5.154 (B72), CN6.154 (B72), CN7.154 (B72)
- new net B73: CN1.155 (B73), CN2.155 (B73), CN3.155 (B73), CN4.155 (B73), CN5.155 (B73), CN6.155 (B73), CN7.155 (B73)
- new net B74: CN1.156 (B74), CN2.156 (B74), CN3.156 (B74), CN4.156 (B74), CN5.156 (B74), CN6.156 (B74), CN7.156 (B74)
- new net B75: CN1.157 (B75), CN2.157 (B75), CN3.157 (B75), CN4.157 (B75), CN5.157 (B75), CN6.157 (B75), CN7.157 (B75)
- new net B76: CN1.158 (B76), CN2.158 (B76), CN3.158 (B76), CN4.158 (B76), CN5.158 (B76), CN6.158 (B76), CN7.158 (B76)
- new net B77: CN1.159 (B77), CN2.159 (B77), CN3.159 (B77), CN4.159 (B77), CN5.159 (B77), CN6.159 (B77), CN7.159 (B77)
- new net B78: CN1.160 (B78), CN2.160 (B78), CN3.160 (B78), CN4.160 (B78), CN5.160 (B78), CN6.160 (B78), CN7.160 (B78)
- new net B79: CN1.161 (B79), CN2.161 (B79), CN3.161 (B79), CN4.161 (B79), CN5.161 (B79), CN6.161 (B79), CN7.161 (B79)
- new net B8: CN1.90 (B8), CN2.90 (B8), CN3.90 (B8), CN4.90 (B8), CN5.90 (B8), CN6.90 (B8), CN7.90 (B8)
- new net B80: CN1.162 (B80), CN2.162 (B80), CN3.162 (B80), CN4.162 (B80), CN5.162 (B80), CN6.162 (B80), CN7.162 (B80)
- new net B81: CN1.163 (B81), CN2.163 (B81), CN3.163 (B81), CN4.163 (B81), CN5.163 (B81), CN6.163 (B81), CN7.163 (B81)
- new net B82: CN1.164 (B82), CN2.164 (B82), CN3.164 (B82), CN4.164 (B82), CN5.164 (B82), CN6.164 (B82), CN7.164 (B82)
- new net B9: CN1.91 (B9), CN2.91 (B9), CN3.91 (B9), CN4.91 (B9), CN5.91 (B9), CN6.91 (B9), CN7.91 (B9)
Other:
- note added: "BACKPLANE"
- note added: "MOUNTING HOLES"
- company: (none) -> Logan Peterson
- title: (none) -> Santa's Microfactory - Backplane
