File: PCB/Santas Microfactory - State Manager/Santas Microfactory - State Manager.kicad_sch (KiCad schematic)
At the start: 279 parts, among them J1 Conn_01x02, J2 Barrel_Jack, J3 Conn_01x02, J4 Bus_PCI_Express_x16, P1 USB_C_Plug, Q1 NPN, Q10 NPN, Q11 NPN, Q12 NPN, Q13 NPN, Q14 NPN, Q15 NPN, Q16 NPN, Q17 NPN, Q18 NPN, Q19 NPN, Q2 NPN, Q20 NPN, Q21 NPN, Q22 NPN, Q23 NPN, Q24 NPN, Q25 NPN, Q26 NPN, Q27 NPN, Q28 NPN, Q29 NPN, Q3 NPN, Q30 NPN, Q31 NPN, Q32 NPN, Q33 NPN, Q4 NPN, Q5 NPN, Q6 NPN, Q7 NPN, Q8 NPN, Q9 NPN, U1 LM2596SX-5.0/NOPB, U2 LM555xN

Commit message: More work
Connections:
- net +3.3V is gone; now on net +5V: R3.1
- net L0: now also D118.1 (K), Q28.2 (B)
- net L3: now also D119.1 (K), Q29.2 (B)
Changed lines of the file:
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@@
 	(wire
 		(pts
-			(xy 993.14 191.77) (xy 993.14 190.5)
-		)
-		(stroke
-			(width 0)
-			(type default)
-		)
-	)
-	(wire
-		(pts
 			(xy 177.8 146.05) (xy 177.8 144.78)
 		)
@@
 	(wire
 		(pts
+			(xy 955.04 191.77) (xy 956.31 191.77)
+		)
+		(stroke
+			(width 0)
+			(type default)
+		)
+	)
+	(wire
+		(pts
 			(xy 830.58 133.35) (xy 830.58 134.62)
 		)
@@
 	(wire
 		(pts
-			(xy 993.14 191.77) (xy 991.87 191.77)
-		)
-		(stroke
-			(width 0)
-			(type default)
-		)
-	)
-	(wire
-		(pts
 			(xy 431.8 163.83) (xy 453.39 163.83)
 		)
@@
 	(wire
 		(pts
+			(xy 955.04 190.5) (xy 955.04 191.77)
+		)
+		(stroke
+			(width 0)
+			(type default)
+		)
+	)
+	(wire
+		(pts
 			(xy 377.19 171.45) (xy 377.19 172.72)
 		)
@@
 		)
 	)
-	(global_label "SEED_0"
-		(shape input)
-		(at 991.87 191.77 180)
-		(fields_autoplaced yes)
-		(effects
-			(font
-				(size 1.27 1.27)
-			)
-			(justify right)
-		)
-		(property "Intersheetrefs" "${INTERSHEET_REFS}"
-			(at 981.9302 191.77 0)
-			(effects
-				(font
-					(size 1.27 1.27)
-				)
-				(justify right)
-				(hide yes)
-			)
-		)
-	)
 	(global_label "TAP_G9"
 		(shape input)
@@
 		)
 	)
+	(global_label "L3"
+		(shape input)
+		(at 449.58 251.46 180)
+		(fields_autoplaced yes)
+		(effects
+			(font
+				(size 1.27 1.27)
+			)
+			(justify right)
+		)
+		(property "Intersheetrefs" "${INTERSHEET_REFS}"
+			(at 444.3572 251.46 0)
+			(effects
+				(font
+					(size 1.27 1.27)
+				)
+				(justify right)
+				(hide yes)
+			)
+		)
+	)
 	(global_label "TAP_C5"
 		(shape input)
@@
 	(global_label "L0"
 		(shape input)
-		(at 21.59 229.87 180)
+		(at 426.72 251.46 180)
 		(fields_autoplaced yes)
 		(effects
@@
 		)
 		(property "Intersheetrefs" "${INTERSHEET_REFS}"
-			(at 16.3672 229.87 0)
+			(at 421.4972 251.46 0)
 			(effects
 				(font
@@
 		)
 	)
-	(global_label "INPUT5"
+	(global_label "L0"
 		(shape input)
-		(at 1282.7 240.03 180)
+		(at 21.59 229.87 180)
 		(fields_autoplaced yes)
 		(effects
@@
 		)
 		(property "Intersheetrefs" "${INTERSHEET_REFS}"
-			(at 1273.0019 240.03 0)
+			(at 16.3672 229.87 0)
 			(effects
 				(font
@@
 		)
 	)
-	(global_label "NRESET"
+	(global_label "INPUT5"
 		(shape input)
-		(at 723.9 133.35 180)
+		(at 1282.7 240.03 180)
 		(fields_autoplaced yes)
 		(effects
@@
 		)
 		(property "Intersheetrefs" "${INTERSHEET_REFS}"
-			(at 713.8392 133.35 0)
+			(at 1273.0019 240.03 0)
 			(effects
 				(font
@@
 		)
 	)
-	(global_label "NCLK"
+	(global_label "NRESET"
 		(shape input)
-		(at 1282.7 151.13 180)
+		(at 723.9 133.35 180)
 		(fields_autoplaced yes)
 		(effects
@@
 		)
 		(property "Intersheetrefs" "${INTERSHEET_REFS}"
-			(at 1274.8162 151.13 0)
+			(at 713.8392 133.35 0)
 			(effects
 				(font
@@
 		)
 	)
-	(global_label "TAP_G8"
+	(global_label "NCLK"
 		(shape input)
-		(at 1282.7 201.93 180)
+		(at 1282.7 151.13 180)
 		(fields_autoplaced yes)
 		(effects
@@
 		)
 		(property "Intersheetrefs" "${INTERSHEET_REFS}"
-			(at 1272.9415 201.93 0)
+			(at 1274.8162 151.13 0)
 			(effects
 				(font
@@
 		)
 	)
-	(global_label "SEED_0"
+	(global_label "TAP_G8"
 		(shape input)
-		(at 956.31 191.77 180)
+		(at 1282.7 201.93 180)
 		(fields_autoplaced yes)
 		(effects
@@
 		)
 		(property "Intersheetrefs" "${INTERSHEET_REFS}"
-			(at 946.3702 191.77 0)
+			(at 1272.9415 201.93 0)
 			(effects
 				(font
@@
 	(symbol
 		(lib_id "power:+5V")
-		(at 993.14 190.5 0)
+		(at 955.04 190.5 0)
 		(unit 1)
 		(exclude_from_sim no)
@@
 		(on_board yes)
 		(dnp no)
-		(fields_autoplaced yes)
 		(property "Reference" "#PWR0122"
-			(at 993.14 194.31 0)
+			(at 955.04 194.31 0)
 			(effects
 				(font
@@
 		)
 		(property "Value" "+5V"
-			(at 993.14 185.42 0)
+			(at 951.484 188.976 0)
 			(effects
 				(font
@@
 		)
 		(property "Footprint" ""
-			(at 993.14 190.5 0)
+			(at 955.04 190.5 0)
 			(effects
 				(font
@@
 		)
 		(property "Datasheet" ""
-			(at 993.14 190.5 0)
+			(at 955.04 190.5 0)
 			(effects
 				(font
@@
 		)
 		(property "Description" "Power symbol creates a global label with name \"+5V\""
-			(at 993.14 190.5 0)
+			(at 955.04 190.5 0)
 			(effects
 				(font
@@
 	)
 	(symbol
-		(lib_id "power:+3.3V")
-		(at 132.08 83.82 0)
-		(unit 1)
-		(exclude_from_sim no)
-		(in_bom yes)
-		(on_board yes)
-		(dnp no)
-		(property "Reference" "#PWR013"
-			(at 132.08 87.63 0)
-			(effects
-				(font
-					(size 1.27 1.27)
-				)
-				(hide yes)
-			)
-		)
-		(property "Value" "+3.3V"
-			(at 135.636 83.058 0)
-			(effects
-				(font
-					(size 1.27 1.27)
-				)
-			)
-		)
-		(property "Footprint" ""
-			(at 132.08 83.82 0)
-			(effects
-				(font
-					(size 1.27 1.27)
-				)
-				(hide yes)
-			)
-		)
-		(property "Datasheet" ""
-			(at 132.08 83.82 0)
-			(effects
-				(font
-					(size 1.27 1.27)
-				)
-				(hide yes)
-			)
-		)
-		(property "Description" "Power symbol creates a global label with name \"+3.3V\""
-			(at 132.08 83.82 0)
-			(effects
-				(font
-					(size 1.27 1.27)
-				)
-				(hide yes)
-			)
-		)
-		(pin "1"
-		)
-		(instances
-			(project "Santas Microfactory - State Manager"
-				(path "/78807986-50ca-41b8-b1ce-82f3b61b40aa"
-					(reference "#PWR013")
-					(unit 1)
-				)
-			)
-		)
-	)
-	(symbol
 		(lib_id "Device:R")
 		(at 872.49 149.86 0)
@@
 					(unit 1)
 				)
+			)
+		)
+	)
+	(symbol
+		(lib_id "power:+5V")
+		(at 132.08 83.82 0)
+		(unit 1)
+		(exclude_from_sim no)
+		(in_bom yes)
+		(on_board yes)
+		(dnp no)
+		(fields_autoplaced yes)
+		(property "Reference" "#PWR013"
+			(at 132.08 87.63 0)
+			(effects
+				(font
+					(size 1.27 1.27)
+				)
+				(hide yes)
+			)
+		)
+		(property "Value" "+5V"
+			(at 132.08 78.74 0)
+			(effects
+				(font
+					(size 1.27 1.27)
+				)
+			)
+		)
+		(property "Footprint" ""
+			(at 132.08 83.82 0)
+			(effects
+				(font
+					(size 1.27 1.27)
+				)
+				(hide yes)
+			)
+		)
+		(property "Datasheet" ""
+			(at 132.08 83.82 0)
+			(effects
+				(font
+					(size 1.27 1.27)
+				)
+				(hide yes)
+			)
+		)
+		(property "Description" "Power symbol creates a global label with name \"+5V\""
+			(at 132.08 83.82 0)
+			(effects
+				(font
+					(size 1.27 1.27)
+				)
+				(hide yes)
+			)
+		)
+		(pin "1"
+		)
+		(instances
+			(project "Santas Microfactory - State Manager"
+				(path "/78807986-50ca-41b8-b1ce-82f3b61b40aa"
+					(reference "#PWR013")
+					(unit 1)
+				)
