File: PCB/Santas Microfactory - State Manager/Santas Microfactory - State Manager.kicad_pcb (KiCad board)
At the start: 2 copper layers, 200 x 191.1 mm, 279 parts, among them J1 Conn_01x02, J2 Barrel_Jack, J3 Conn_01x02, J4 Bus_PCI_Express_x16, P1 USB_C_Plug, Q1 NPN, Q10 NPN, Q11 NPN, Q12 NPN, Q13 NPN, Q14 NPN, Q15 NPN, Q16 NPN, Q17 NPN, Q18 NPN, Q19 NPN, Q2 NPN, Q20 NPN, Q21 NPN, Q22 NPN, Q23 NPN, Q24 NPN, Q25 NPN, Q26 NPN, Q27 NPN, Q28 NPN, Q29 NPN, Q3 NPN, Q30 NPN, Q31 NPN, Q32 NPN, Q33 NPN, Q4 NPN, Q5 NPN, Q6 NPN, Q7 NPN, Q8 NPN, Q9 NPN, U1 LM2596SX-5.0/NOPB, U2 LM555xN

Commit message: More work
Parts:
- moved D21 328.3 mm to (235.2, 102.5)
- moved D20 322.4 mm to (229.0, 102.5)
- moved D41 321.9 mm to (235.2, 107.0)
- moved J2 320.6 mm to (221.2, 69.8), turned to -90 degrees
- moved D3 320.5 mm to (232.3, 60.5), turned to 180 degrees
- moved D40 315.5 mm to (228.7, 107.0)
- moved D19 310.0 mm to (216.2, 102.5)
- moved D77 309.6 mm to (235.1, 111.5)
- moved J3 308.6 mm to (239.2, 71.8), turned to 180 degrees
- moved D67 305.3 mm to (228.6, 111.5)
- moved D18 304.1 mm to (210.0, 102.5)
- moved J1 304.1 mm to (230.0, 71.8), turned to 180 degrees
- moved D39 303.3 mm to (216.3, 107.0)
- moved D102 299.1 mm to (235.1, 116.0)
- moved D1 297.9 mm to (199.2, 77.7), turned to 180 degrees
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Connections:
- D1 pad 1: SEED_0 -> +5V
- D113 pad 1: SEED_0 -> +5V
- D118 pad 1: Net-(D118-K) -> L0
- D119 pad 1: Net-(D119-K) -> L3
- D125 pad 1: SEED_0 -> +5V
- J4 pad A10: SEED_0 -> +5V
- J4 pad A2: SEED_0 -> +5V
- J4 pad A3: SEED_0 -> +5V
- J4 pad A9: SEED_0 -> +5V
- J4 pad B1: SEED_0 -> +5V
- J4 pad B10: SEED_0 -> +5V
- J4 pad B2: SEED_0 -> +5V
- J4 pad B3: SEED_0 -> +5V
- J4 pad B8: SEED_0 -> +5V
- P1 pad A4: SEED_0 -> +5V
- P1 pad A9: SEED_0 -> +5V
- P1 pad B4: SEED_0 -> +5V
- P1 pad B9: SEED_0 -> +5V
- Q28 pad 2: Net-(D118-K) -> L0
- Q29 pad 2: Net-(D119-K) -> L3
- R10 pad 1: SEED_0 -> +5V
- R11 pad 1: SEED_0 -> +5V
- R12 pad 1: SEED_0 -> +5V
- R13 pad 1: SEED_0 -> +5V
- R14 pad 1: SEED_0 -> +5V
- R15 pad 1: SEED_0 -> +5V
- R16 pad 1: SEED_0 -> +5V
- R17 pad 1: SEED_0 -> +5V
- R18 pad 1: SEED_0 -> +5V
- R19 pad 1: SEED_0 -> +5V
- R20 pad 1: SEED_0 -> +5V
- R21 pad 1: SEED_0 -> +5V
- R22 pad 1: SEED_0 -> +5V
- R23 pad 1: SEED_0 -> +5V
- R24 pad 1: SEED_0 -> +5V
- R25 pad 1: SEED_0 -> +5V
- R26 pad 1: SEED_0 -> +5V
- R27 pad 1: SEED_0 -> +5V
- R28 pad 1: SEED_0 -> +5V
- R29 pad 1: SEED_0 -> +5V
- R3 pad 1: +3.3V -> +5V
- R30 pad 1: SEED_0 -> +5V
- R31 pad 1: SEED_0 -> +5V
- R32 pad 1: SEED_0 -> +5V
- R33 pad 1: SEED_0 -> +5V
- R34 pad 1: SEED_0 -> +5V
- R35 pad 1: SEED_0 -> +5V
- R36 pad 1: SEED_0 -> +5V
- R37 pad 1: SEED_0 -> +5V
- R38 pad 1: SEED_0 -> +5V
- R39 pad 1: SEED_0 -> +5V
- R4 pad 1: SEED_0 -> +5V
- R40 pad 1: SEED_0 -> +5V
- R41 pad 1: SEED_0 -> +5V
- R42 pad 1: SEED_0 -> +5V
- R43 pad 1: SEED_0 -> +5V
- R49 pad 1: SEED_0 -> +5V
- R5 pad 1: SEED_0 -> +5V
- R50 pad 1: SEED_0 -> +5V
- R51 pad 1: SEED_0 -> +5V
- R52 pad 1: SEED_0 -> +5V
- R53 pad 1: SEED_0 -> +5V
- R54 pad 1: SEED_0 -> +5V
- R55 pad 1: SEED_0 -> +5V
- R56 pad 1: SEED_0 -> +5V
- R57 pad 1: SEED_0 -> +5V
- R58 pad 1: SEED_0 -> +5V
- R59 pad 1: SEED_0 -> +5V
- R6 pad 1: SEED_0 -> +5V
- R60 pad 1: SEED_0 -> +5V
- R61 pad 1: SEED_0 -> +5V
- R62 pad 1: SEED_0 -> +5V
- R63 pad 1: SEED_0 -> +5V
- R64 pad 1: SEED_0 -> +5V
- R65 pad 1: SEED_0 -> +5V
- R66 pad 1: SEED_0 -> +5V
- R67 pad 1: SEED_0 -> +5V
- R68 pad 1: SEED_0 -> +5V
- R69 pad 1: SEED_0 -> +5V
- R7 pad 1: SEED_0 -> +5V
- R70 pad 1: SEED_0 -> +5V
- R71 pad 1: SEED_0 -> +5V
- R72 pad 1: SEED_0 -> +5V
- R73 pad 1: SEED_0 -> +5V
- R74 pad 1: SEED_0 -> +5V
- R75 pad 1: SEED_0 -> +5V
- R76 pad 1: SEED_0 -> +5V
- R77 pad 1: SEED_0 -> +5V
- R78 pad 1: SEED_0 -> +5V
- R79 pad 1: SEED_0 -> +5V
- R8 pad 1: SEED_0 -> +5V
- R80 pad 1: SEED_0 -> +5V
- R81 pad 1: SEED_0 -> +5V
- R82 pad 1: SEED_0 -> +5V
- R83 pad 1: SEED_0 -> +5V
- R84 pad 1: SEED_0 -> +5V
- R85 pad 1: SEED_0 -> +5V
- R86 pad 1: SEED_0 -> +5V
- R87 pad 1: SEED_0 -> +5V
- R88 pad 1: SEED_0 -> +5V
- R89 pad 1: SEED_0 -> +5V
- R9 pad 1: SEED_0 -> +5V
- R91 pad 1: SEED_0 -> +5V
- R92 pad 1: SEED_0 -> +5V
- R93 pad 1: SEED_0 -> +5V
- R94 pad 1: SEED_0 -> +5V
- R95 pad 1: SEED_0 -> +5V
- R96 pad 1: SEED_0 -> +5V
- R97 pad 1: SEED_0 -> +5V
- R98 pad 1: SEED_0 -> +5V
- R99 pad 1: SEED_0 -> +5V
- U2 pad 4: SEED_0 -> +5V
- U2 pad 8: SEED_0 -> +5V
Routing:
- net +5V: track 0.00 -> 907.4 mm, vias 0 -> 1
- net NCLK: track 0.00 -> 412.7 mm
- net CLK: track 0.00 -> 390.3 mm
- net SEED_1: track 0.00 -> 303.0 mm
- net L3: track 0.00 -> 296.8 mm
- net L0: track 0.00 -> 293.3 mm, vias 0 -> 4
- net NRESET: track 0.00 -> 284.3 mm, vias 0 -> 2
- net RESET: track 0.00 -> 275.0 mm, vias 0 -> 7
- net L1: track 0.00 -> 155.0 mm, vias 0 -> 2
- net SEED_3: track 0.00 -> 152.1 mm, vias 0 -> 8
- net SEED_2: track 0.00 -> 134.7 mm
- net SEED_4: track 0.00 -> 93.5 mm, vias 0 -> 4
- net RAW_CLK: track 0.00 -> 93.5 mm
- net NHALT: track 0.00 -> 80.0 mm
- net REG_BATT+: track 0.00 -> 59.0 mm
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- added copper zone on B.Cu, net GND
- added copper zone on F.Cu, net GND
Other:
- board size 200 x 191.1 mm -> 200 x 101 mm

Commit message: All silkscreen additions + Gerbers and CAD files
Silkscreen and Gerbers are done, but I plan on using the CAD to create additional renders.
Parts:
- added G***: LOGO, LOGO, F.Cu at (222.0, 85.0)
- added G***: LOGO, LOGO, F.Cu at (97.0, 100.8)
- added G***: LOGO, LOGO, F.Cu at (65.8, 146.2)
- added G***: LOGO, LOGO, F.Cu at (65.6, 105.1)
Other:
- board text added: "Designed by: Logan Peterson"
- board text added: "State Manager"
