File: PCB/Santas Microfactory Master/Santas Microfactory Master.kicad_sch (KiCad schematic)
At the start: 0 parts

Commit message: Chutes Done + Main Conveyor Layout
Other:
- note added: "TODO: Input Output board Input Chutes board Input Main Conveyor board"
- note removed: "TODO: Board Connector"
Changed lines of the file:
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@@
 		(company "Logan Peterson")
 	)
-	(text "TODO:\nBoard Connector"
+	(text "TODO:\nInput Output board\nInput Chutes board\nInput Main Conveyor board\n"
 		(exclude_from_sim no)
-		(at -141.478 46.482 0)
+		(at 11.43 -55.88 0)
 		(effects
 			(font
