File: PCB/Santas Microfactory - Main Conveyor/Santas Microfactory - Main Conveyor.kicad_pcb (KiCad board)
At the start: 4 copper layers, 200 x 191.1 mm, 179 parts, among them J1 Bus_PCI_Express_x16, J2 Conn_01x10_Pin, J3 Conn_01x10_Pin, Q1 NPN, Q10 NPN, Q11 NPN, Q12 NPN, Q13 NPN, Q14 NPN, Q15 NPN, Q16 NPN, Q17 NPN, Q18 NPN, Q19 NPN, Q2 NPN, Q20 NPN, Q21 NPN, Q22 NPN, Q23 NPN, Q24 NPN, Q3 NPN, Q4 NPN, Q5 NPN, Q6 NPN, Q7 NPN, Q8 NPN, Q9 NPN

Commit message: Update Input Output Board
Parts:
- added J4: Conn_01x06_Pin, Connector_PinHeader_2.54mm:PinHeader_1x06_P2.54mm_Horizontal, F.Cu at (119.7, 221.8)
Routing:
- net LOAD4: track 277.6 -> 364.6 mm
- net LOAD3: track 308.6 -> 383.5 mm
- net LOAD0: track 165.1 -> 239.1 mm, vias 1 -> 2
- net LOAD1: track 196.4 -> 253.3 mm
- net LOAD2: track 310.2 -> 354.6 mm
- net LOAD5: track 300.4 -> 312.3 mm
- net OUT_C7: track 253.9 -> 259.4 mm
- net TAP_G6: track 676.8 -> 678.4 mm
- net TAP_G8: track 627.3 -> 628.6 mm
- net TAP_G9: track 461.2 -> 462.2 mm
- net OUT_G7: track 362.5 -> 363.3 mm
- net TAP_G2: track 531.7 -> 532.5 mm
- net OUT_G1: track 416.5 -> 417.3 mm
- net TAP_G3: track 614.1 -> 614.9 mm
- net OUT_G4: track 404.9 -> 405.7 mm
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