File: PCB/Santas Microfactory - Main Conveyor/Santas Microfactory - Main Conveyor.kicad_pcb (KiCad board)
At the start: 4 copper layers, 200 x 191.1 mm, 180 parts, among them J1 Bus_PCI_Express_x16, J2 Conn_01x10_Pin, J3 Conn_01x10_Pin, J4 Conn_01x06_Pin, Q1 NPN, Q10 NPN, Q11 NPN, Q12 NPN, Q13 NPN, Q14 NPN, Q15 NPN, Q16 NPN, Q17 NPN, Q18 NPN, Q19 NPN, Q2 NPN, Q20 NPN, Q21 NPN, Q22 NPN, Q23 NPN, Q24 NPN, Q3 NPN, Q4 NPN, Q5 NPN, Q6 NPN, Q7 NPN, Q8 NPN, Q9 NPN

Commit message: All silkscreen additions + Gerbers and CAD files
Silkscreen and Gerbers are done, but I plan on using the CAD to create additional renders.
Parts:
- added G***: LOGO, LOGO, F.Cu at (108.8, 213.2)
Other:
- board text added: "COAL CONVEYOR"
- board text added: "Designed by: Logan Peterson"
- board text added: "GIFT CONVEYOR"
- board text added: "INPUT"
- board text added: "Main Conveyor"
