File: PCB/Santas Microfactory - Main Conveyor/Santas Microfactory - Main Conveyor.kicad_sch (KiCad schematic)
At the start: 0 parts

Commit message: Chutes Done + Main Conveyor Layout
Parts:
- added D1, D10, D11, D12, D13, D14, D15, D16, D17, D18, D19, D2, D20, D21, D22, D23, D24, D25, D26, D27, D28, D29, D3, D30, D31, D32, D33, D34, D35, D36, D37, D38, D39, D4, D40, D41, D42, D43, D44, D45, D46, D47, D48, D49, D5, D50, D51, D52, D53, D54, D55, D56, D57, D58, D59, D6, D60, D61, D62, D63, D64, D65, D66, D67, D68, D69, D7, D70, D71, D72, D8, D9: D, Diode_THT:D_DO-35_SOD27_P2.54mm_Vertical_AnodeUp, symbol Device:D
- added DFF1, DFF10, DFF11, DFF12, DFF13, DFF14, DFF15, DFF16, DFF17, DFF18, DFF19, DFF2, DFF20, DFF3, DFF4, DFF5, DFF6, DFF7, DFF8, DFF9: ~, shenanigans:DFF-shenanigans, symbol shenanigans:DFF-shenanigans
- added J1: Bus_PCI_Express_x16, Connector_PCBEdge:BUS_PCIexpress_x16, symbol Connector:Bus_PCI_Express_x16
- added J2, J3: Conn_01x10_Pin, Connector_PinHeader_2.54mm:PinHeader_1x10_P2.54mm_Horizontal, symbol Connector:Conn_01x10_Pin
- added Q1, Q10, Q11, Q12, Q13, Q14, Q15, Q16, Q17, Q18, Q19, Q2, Q20, Q21, Q22, Q23, Q24, Q3, Q4, Q5, Q6, Q7, Q8, Q9: NPN, Package_TO_SOT_THT:TO-92L_Inline, symbol Simulation_SPICE:NPN
- added R1, R10, R11, R12, R13, R14, R15, R16, R17, R18, R19, R2, R20, R21, R22, R23, R24, R25, R26, R27, R28, R29, R3, R30, R31, R32, R33, R34, R35, R36, R37, R38, R39, R4, R40, R41, R42, R43, R44, R45, R46, R47, R48, R49, R5, R50, R51, R52, R53, R54, R55, R56, R57, R58, R59, R6, R60, R7, R8, R9: 10k, Resistor_THT:R_Axial_DIN0207_L6.3mm_D2.5mm_P2.54mm_Vertical, symbol Device:R
Connections:
- new net: D52.1 (K), DFF7.16 (DOUT)
- new net: D37.2 (A), D43.2 (A), Q13.2 (B), R43.2
- new net: D14.1 (K), D2.1 (K), D8.1 (K), R9.2
- new net: D48.1 (K), Q24.1 (C), R42.2
- new net: D27.2 (A), D33.2 (A), Q9.2 (B), R27.2
- new net: D65.1 (K), DFF19.16 (DOUT)
- new net: D42.2 (A), D48.2 (A), Q18.2 (B), R48.2
- new net: D51.1 (K), DFF6.16 (DOUT)
- new net: D40.2 (A), D46.2 (A), Q16.2 (B), R46.2
- new net: D45.1 (K), Q21.1 (C), R39.2
- new net: D28.2 (A), D34.2 (A), Q10.2 (B), R28.2
- new net: D47.1 (K), Q23.1 (C), R41.2
- new net: D1.1 (K), D13.1 (K), D7.1 (K), R7.2
- new net: D11.1 (K), D17.1 (K), D5.1 (K), R15.1
- new net: D25.2 (A), D31.2 (A), Q7.2 (B), R25.2
- new net: D53.1 (K), DFF9.16 (DOUT)
- new net: D39.2 (A), D45.2 (A), Q15.2 (B), R45.2
- new net: D43.1 (K), Q19.1 (C), R37.2
- new net: D29.2 (A), D35.2 (A), Q11.2 (B), R29.2
- new net: D12.1 (K), D18.1 (K), D6.1 (K), R17.1
- new net: D10.1 (K), D16.1 (K), D4.1 (K), R13.1
- new net: D44.1 (K), Q20.1 (C), R38.2
- new net: D63.1 (K), DFF16.16 (DOUT)
- new net: D15.1 (K), D3.1 (K), D9.1 (K), R11.1
- new net: D38.2 (A), D44.2 (A), Q14.2 (B), R44.2
- new net: D49.1 (K), DFF3.16 (DOUT)
- new net: D46.1 (K), Q22.1 (C), R40.2
- new net: D61.1 (K), DFF13.16 (DOUT)
- new net: D26.2 (A), D32.2 (A), Q8.2 (B), R26.2
- new net: D41.2 (A), D47.2 (A), Q17.2 (B), R47.2
- new net: D30.2 (A), D36.2 (A), Q12.2 (B), R30.2
- new net: D50.1 (K), DFF4.16 (DOUT)
- new net: D62.1 (K), DFF14.16 (DOUT)
- new net: D64.1 (K), DFF17.16 (DOUT)
- new net +5V: DFF1.10 (5V), DFF10.10 (5V), DFF11.10 (5V), DFF12.10 (5V), DFF13.10 (5V), DFF14.10 (5V), DFF15.10 (5V), DFF16.10 (5V), DFF17.10 (5V), DFF18.10 (5V), DFF19.10 (5V), DFF2.10 (5V), DFF20.10 (5V), DFF3.10 (5V), DFF4.10 (5V), DFF5.10 (5V), DFF6.10 (5V), DFF7.10 (5V), DFF8.10 (5V), DFF9.10 (5V), J1.A10 (+3.3V), J1.A2 (+12V), J1.A3 (+12V), J1.A9 (+3.3V), J1.B1 (+12V), J1.B10 (3.3Vaux), J1.B2 (+12V), J1.B3 (+12V), J1.B8 (+3.3V), R1.1, R10.1, R12.1, R14.1, R16.1, R18.1, R19.1, R2.1, R20.1, R21.1, R22.1, R23.1, R24.1, R25.1, R26.1, R27.1, R28.1, R29.1, R3.1, R30.1, R31.1, R32.1, R33.1, R34.1, R35.1, R36.1, R37.1, R38.1, R39.1, R4.1, R40.1, R41.1, R42.1, R43.1, R44.1, R45.1, R46.1, R47.1, R48.1, R49.1, R5.1, R50.1, R51.1, R52.1, R53.1, R54.1, R55.1, R56.1, R57.1, R58.1, R59.1, R6.1, R60.1, R8.1
- new net CLK: DFF1.14 (CLK), DFF10.14 (CLK), DFF11.14 (CLK), DFF12.14 (CLK), DFF13.14 (CLK), DFF14.14 (CLK), DFF15.14 (CLK), DFF16.14 (CLK), DFF17.14 (CLK), DFF18.14 (CLK), DFF19.14 (CLK), DFF2.14 (CLK), DFF20.14 (CLK), DFF3.14 (CLK), DFF4.14 (CLK), DFF5.14 (CLK), DFF6.14 (CLK), DFF7.14 (CLK), DFF8.14 (CLK), DFF9.14 (CLK), J1.A13 (REFCLK+)
- new net CLK_TICK: J1.A1 (~{PRSNT1}), Q19.2 (B), Q20.2 (B), Q21.2 (B), Q22.2 (B), Q23.2 (B), Q24.2 (B)
- new net CORR_0: J1.B82 (RSVD)
- new net CORR_1: J1.A50 (RSVD)
- new net CORR_2: J1.A33 (RSVD)
- new net CORR_3: J1.B30 (RSVD)
- new net CORR_4: J1.A32 (RSVD)
- new net CORR_5: J1.A19 (RSVD)
- new net GND: DFF1.11 (GND), DFF10.11 (GND), DFF11.11 (GND), DFF12.11 (GND), DFF13.11 (GND), DFF14.11 (GND), DFF15.11 (GND), DFF16.11 (GND), DFF17.11 (GND), DFF18.11 (GND), DFF19.11 (GND), DFF2.11 (GND), DFF20.11 (GND), DFF3.11 (GND), DFF4.11 (GND), DFF5.11 (GND), DFF6.11 (GND), DFF7.11 (GND), DFF8.11 (GND), DFF9.11 (GND), J1.A12 (GND), J1.A15 (GND), J1.A18 (GND), J1.A20 (GND), J1.A23 (GND), J1.A24 (GND), J1.A27 (GND), J1.A28 (GND), J1.A31 (GND), J1.A34 (GND), J1.A37 (GND), J1.A38 (GND), J1.A4 (GND), J1.A41 (GND), J1.A42 (GND), J1.A45 (GND), J1.A46 (GND), J1.A49 (GND), J1.A51 (GND), J1.A54 (GND), J1.A55 (GND), J1.A58 (GND), J1.A59 (GND), J1.A62 (GND), J1.A63 (GND), J1.A66 (GND), J1.A67 (GND), J1.A70 (GND), J1.A71 (GND), J1.A74 (GND), J1.A75 (GND), J1.A78 (GND), J1.A79 (GND), J1.A82 (GND), J1.B13 (GND), J1.B16 (GND), J1.B18 (GND), J1.B21 (GND), J1.B22 (GND), J1.B25 (GND), J1.B26 (GND), J1.B29 (GND), J1.B32 (GND), J1.B35 (GND), J1.B36 (GND), J1.B39 (GND), J1.B4 (GND), J1.B40 (GND), J1.B43 (GND), J1.B44 (GND), J1.B47 (GND), J1.B49 (GND), J1.B52 (GND), J1.B53 (GND), J1.B56 (GND), J1.B57 (GND), J1.B60 (GND), J1.B61 (GND), J1.B64 (GND), J1.B65 (GND), J1.B68 (GND), J1.B69 (GND), J1.B7 (GND), J1.B72 (GND), J1.B73 (GND), J1.B76 (GND), J1.B77 (GND), J1.B80 (GND), Q1.3 (E), Q10.3 (E), Q11.3 (E), Q12.3 (E), Q13.3 (E), Q14.3 (E), Q15.3 (E), Q16.3 (E), Q17.3 (E), Q18.3 (E), Q19.3 (E), Q2.3 (E), Q20.3 (E), Q21.3 (E), Q22.3 (E), Q23.3 (E), Q24.3 (E), Q3.3 (E), Q4.3 (E), Q5.3 (E), Q6.3 (E), Q7.3 (E), Q8.3 (E), Q9.3 (E), R11.2, R13.2, R15.2, R17.2, R7.1, R9.1
- new net HALT: J1.B48 (~{PRSNT2})
- new net INPUT0: D25.1 (K), J1.B62 (PETp11)
- new net INPUT1: D26.1 (K), J1.B63 (PETn11)
- new net INPUT2: D27.1 (K), J1.B66 (PETp12)
- new net INPUT3: D28.1 (K), J1.B67 (PETn12)
- new net INPUT4: D29.1 (K), J1.B70 (PETp13)
- new net INPUT5: D30.1 (K), J1.B71 (PETn13)
- new net IN_C0: DFF11.13 (DIN), J1.B6 (SMDAT)
- new net IN_G0: DFF1.13 (DIN), J1.B5 (SMCLK)
- new net LOAD0: D10.2 (A), D11.2 (A), D12.2 (A), D19.2 (A), D20.2 (A), D21.2 (A), D22.2 (A), D23.2 (A), D24.2 (A), D7.2 (A), D8.2 (A), D9.2 (A), J1.B50 (PETp8), Q1.2 (B), Q2.2 (B), Q3.2 (B), Q4.2 (B), Q5.2 (B), Q6.2 (B), R10.2, R12.2, R14.2, R16.2, R18.2, R8.2
- new net LOAD1: J1.B51 (PETn8)
- new net LOAD2: J1.B54 (PETp9)
- new net LOAD3: J1.B55 (PETn9)
- new net LOAD4: J1.B58 (PETp10)
- new net LOAD5: J1.B59 (PETn10)
- new net NCLK: DFF1.15 (NCLK), DFF10.15 (NCLK), DFF11.15 (NCLK), DFF12.15 (NCLK), DFF13.15 (NCLK), DFF14.15 (NCLK), DFF15.15 (NCLK), DFF16.15 (NCLK), DFF17.15 (NCLK), DFF18.15 (NCLK), DFF19.15 (NCLK), DFF2.15 (NCLK), DFF20.15 (NCLK), DFF3.15 (NCLK), DFF4.15 (NCLK), DFF5.15 (NCLK), DFF6.15 (NCLK), DFF7.15 (NCLK), DFF8.15 (NCLK), DFF9.15 (NCLK), J1.A14 (REFCLK-)
- new net NHALT: J1.B81 (~{PRSNT2})
- new net NLOAD0: D55.1 (K), D67.1 (K), Q1.1 (C), Q2.1 (C), Q3.1 (C), Q4.1 (C), Q5.1 (C), Q6.1 (C), R1.2, R2.2, R3.2, R4.2, R5.2, R6.2
- new net NLOAD1: D56.1 (K), D68.1 (K)
- new net NLOAD2: D57.1 (K), D69.1 (K)
- new net NLOAD3: D58.1 (K), D70.1 (K)
- new net NLOAD4: D59.1 (K), D71.1 (K)
- new net NLOAD5: D60.1 (K), D72.1 (K)
- new net NOUT _C0: DFF11.17 (NDOUT)
- new net NOUT _C1: DFF12.17 (NDOUT)
- new net NOUT _C2: DFF13.17 (NDOUT)
- new net NOUT _C3: DFF14.17 (NDOUT)
- new net NOUT _C4: DFF15.17 (NDOUT)
- new net NOUT _C5: DFF16.17 (NDOUT)
- new net NOUT _C6: DFF17.17 (NDOUT)
- new net NOUT _C7: DFF18.17 (NDOUT)
- new net NOUT _C8: DFF19.17 (NDOUT)
- new net NOUT _C9: DFF20.17 (NDOUT)
- new net NOUT_G0: DFF1.17 (NDOUT)
- new net NOUT_G1: DFF2.17 (NDOUT)
- new net NOUT_G2: DFF3.17 (NDOUT)
- new net NOUT_G3: DFF4.17 (NDOUT)
- new net NOUT_G4: DFF5.17 (NDOUT)
- new net NOUT_G5: DFF6.17 (NDOUT)
- new net NOUT_G6: DFF7.17 (NDOUT)
- new net NOUT_G7: DFF8.17 (NDOUT)
- new net NOUT_G8: DFF9.17 (NDOUT)
- new net NOUT_G9: DFF10.17 (NDOUT)
- new net NREQ0: D31.1 (K), Q13.1 (C), R31.2
- new net NREQ1: D32.1 (K), Q14.1 (C), R32.2
- new net NREQ2: D33.1 (K), Q15.1 (C), R33.2
- new net NREQ3: D34.1 (K), Q16.1 (C), R34.2
- new net NREQ4: D35.1 (K), Q17.1 (C), R35.2
- new net NREQ5: D36.1 (K), Q18.1 (C), R36.2
- new net NRESET: DFF1.12 (NRST), DFF10.12 (NRST), DFF11.12 (NRST), DFF12.12 (NRST), DFF13.12 (NRST), DFF14.12 (NRST), DFF15.12 (NRST), DFF16.12 (NRST), DFF17.12 (NRST), DFF18.12 (NRST), DFF19.12 (NRST), DFF2.12 (NRST), DFF20.12 (NRST), DFF3.12 (NRST), DFF4.12 (NRST), DFF5.12 (NRST), DFF6.12 (NRST), DFF7.12 (NRST), DFF8.12 (NRST), DFF9.12 (NRST), J1.B31 (~{PRSNT2})
- new net OUT_C0: DFF11.16 (DOUT), DFF12.13 (DIN), J2.1 (Pin_1)
- new net OUT_C1: DFF12.16 (DOUT), DFF13.13 (DIN), J2.2 (Pin_2)
- new net OUT_C4: DFF15.16 (DOUT), DFF16.13 (DIN), J2.5 (Pin_5)
- new net OUT_C7: DFF18.16 (DOUT), DFF19.13 (DIN), J2.8 (Pin_8)
- new net OUT_C9: D66.2 (A), D72.2 (A), R60.2
- new net OUT_G0: DFF1.16 (DOUT), DFF2.13 (DIN), J3.1 (Pin_1)
- new net OUT_G1: DFF2.16 (DOUT), DFF3.13 (DIN), J3.2 (Pin_2)
- new net OUT_G4: DFF5.16 (DOUT), DFF6.13 (DIN), J3.5 (Pin_5)
- new net OUT_G7: DFF8.16 (DOUT), DFF9.13 (DIN), J3.8 (Pin_8)
- new net OUT_G9: D54.2 (A), D60.2 (A), R54.2
- new net REQ0: D19.1 (K), D20.1 (K), D21.1 (K), D22.1 (K), D23.1 (K), D24.1 (K), D37.1 (K), Q7.1 (C), R19.2
- new net REQ1: D38.1 (K), Q8.1 (C), R20.2
- new net REQ2: D39.1 (K), Q9.1 (C), R21.2
- new net REQ3: D40.1 (K), Q10.1 (C), R22.2
- new net REQ4: D41.1 (K), Q11.1 (C), R23.2
- new net REQ5: D42.1 (K), Q12.1 (C), R24.2
- new net RESET: J1.B17 (~{PRSNT2})
- new net SEED_1: J1.B14 (PETp0)
- new net SEED_2: J1.B15 (PETn0)
- new net SEED_3: J1.B19 (PETp1)
- new net SEED_4: J1.B20 (PETn1)
- new net TAP_C2: D13.2 (A), D61.2 (A), D67.2 (A), DFF14.13 (DIN), J1.B24 (PETn2), J2.3 (Pin_3), R55.2
- new net TAP_C3: D14.2 (A), D62.2 (A), D68.2 (A), DFF15.13 (DIN), J1.B28 (PETn3), J2.4 (Pin_4), R56.2
- new net TAP_C5: D15.2 (A), D63.2 (A), D69.2 (A), DFF17.13 (DIN), J1.B34 (PETn4), J2.6 (Pin_6), R57.2
- new net TAP_C6: D16.2 (A), D64.2 (A), D70.2 (A), DFF18.13 (DIN), J1.B38 (PETn5), J2.7 (Pin_7), R58.2
- new net TAP_C8: D17.2 (A), D65.2 (A), D71.2 (A), DFF20.13 (DIN), J1.B42 (PETn6), J2.9 (Pin_9), R59.2
- new net TAP_C9: D18.2 (A), D66.1 (K), DFF20.16 (DOUT), J1.B46 (PETn7), J2.10 (Pin_10)
- new net TAP_G2: D1.2 (A), D49.2 (A), D55.2 (A), DFF4.13 (DIN), J1.B23 (PETp2), J3.3 (Pin_3), R49.2
- new net TAP_G3: D2.2 (A), D50.2 (A), D56.2 (A), DFF5.13 (DIN), J1.B27 (PETp3), J3.4 (Pin_4), R50.2
- new net TAP_G5: D3.2 (A), D51.2 (A), D57.2 (A), DFF7.13 (DIN), J1.B33 (PETp4), J3.6 (Pin_6), R51.2
- new net TAP_G6: D4.2 (A), D52.2 (A), D58.2 (A), DFF8.13 (DIN), J1.B37 (PETp5), J3.7 (Pin_7), R52.2
- new net TAP_G8: D5.2 (A), D53.2 (A), D59.2 (A), DFF10.13 (DIN), J1.B41 (PETp6), J3.9 (Pin_9), R53.2
- new net TAP_G9: D54.1 (K), D6.2 (A), DFF10.16 (DOUT), J1.B45 (PETp7), J3.10 (Pin_10)
- new net WRONG_0: J1.B12 (RSVD)
- new net WRONG_1: J1.B11 (~{WAKE})
- new net WRONG_2: J1.A11 (~{PERST})
- new net WRONG_3: J1.B9 (JTAG1)
- new net WRONG_4: J1.A6 (JTAG3)
- new net WRONG_5: J1.A5 (JTAG2), J1.A7 (JTAG4)
Other:
- note added: "AND"
- note added: "COAL CHUTE"
- note added: "GIFT CHUTE"
- note added: "LOAD"
- note added: "MAIN CONVEYOR"
- note added: "NAND"
- note added: "NOT"
- note added: "OR"
- note added: "OUTPUTMASK"
- note added: "SR Latch"
- company: (none) -> Logan Peterson
- title: (none) -> Santa's Microfactory - Main Conveyor

Commit message: Main Conveyor Done
Connections:
- net LOAD0: no longer D10.2 (A), D11.2 (A), D12.2 (A), D20.2 (A), D21.2 (A), D22.2 (A), D23.2 (A), D24.2 (A), D8.2 (A), D9.2 (A), Q2.2 (B), Q3.2 (B), Q4.2 (B), Q5.2 (B), Q6.2 (B), R10.2, R12.2, R14.2, R16.2, R18.2
- net LOAD1: now also D20.2 (A), D8.2 (A), Q2.2 (B), R10.2
- net LOAD2: now also D21.2 (A), D9.2 (A), Q3.2 (B), R12.2
- net LOAD3: now also D10.2 (A), D22.2 (A), Q4.2 (B), R14.2
- net LOAD4: now also D11.2 (A), D23.2 (A), Q5.2 (B), R16.2
- net LOAD5: now also D12.2 (A), D24.2 (A), Q6.2 (B), R18.2
- net NLOAD0: no longer Q2.1 (C), Q3.1 (C), Q4.1 (C), Q5.1 (C), Q6.1 (C), R2.2, R3.2, R4.2, R5.2, R6.2
- net NLOAD1: now also Q2.1 (C), R2.2
- net NLOAD2: now also Q3.1 (C), R3.2
- net NLOAD3: now also Q4.1 (C), R4.2
- net NLOAD4: now also Q5.1 (C), R5.2
- net NLOAD5: now also Q6.1 (C), R6.2
- net REQ0: no longer D20.1 (K), D21.1 (K), D22.1 (K), D23.1 (K), D24.1 (K)
- net REQ1: now also D20.1 (K)
- net REQ2: now also D21.1 (K)
- net REQ3: now also D22.1 (K)
- net REQ4: now also D23.1 (K)
- net REQ5: now also D24.1 (K)
Changed lines of the file:
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@@
 		)
 	)
-	(global_label "LOAD0"
+	(global_label "LOAD4"
 		(shape input)
 		(at 543.56 134.62 0)
@@
 		)
 	)
-	(global_label "NLOAD0"
+	(global_label "NLOAD3"
 		(shape input)
 		(at 438.15 120.65 0)
@@
 		)
 	)
-	(global_label "REQ0"
+	(global_label "REQ2"
 		(shape input)
 		(at 332.74 132.08 180)
@@
 		)
 	)
-	(global_label "LOAD0"
+	(global_label "LOAD2"
 		(shape input)
 		(at 344.17 134.62 0)
@@
 		)
 	)
-	(global_label "REQ0"
+	(global_label "REQ1"
 		(shape input)
 		(at 214.63 132.08 180)
@@
 		)
 	)
-	(global_label "NLOAD0"
+	(global_label "NLOAD2"
 		(shape input)
 		(at 361.95 120.65 0)
@@
 		)
 	)
-	(global_label "LOAD0"
+	(global_label "LOAD1"
 		(shape input)
 		(at 226.06 134.62 0)
@@
 		)
 	)
-	(global_label "REQ0"
+	(global_label "REQ4"
 		(shape input)
 		(at 532.13 132.08 180)
@@
 		)
 	)
-	(global_label "NLOAD0"
+	(global_label "NLOAD4"
 		(shape input)
 		(at 561.34 120.65 0)
@@
 		)
 	)
-	(global_label "REQ0"
+	(global_label "REQ5"
 		(shape input)
 		(at 608.33 132.08 180)
@@
 		)
 	)
-	(global_label "LOAD0"
+	(global_label "LOAD5"
 		(shape input)
 		(at 619.76 134.62 0)
@@
 		)
 	)
-	(global_label "LOAD0"
+	(global_label "LOAD3"
 		(shape input)
 		(at 420.37 134.62 0)
@@
 		)
 	)
-	(global_label "NLOAD0"
+	(global_label "NLOAD5"
 		(shape input)
 		(at 637.54 120.65 0)
@@
 		)
 	)
-	(global_label "NLOAD0"
+	(global_label "NLOAD1"
 		(shape input)
 		(at 243.84 120.65 0)
@@
 		)
 	)
-	(global_label "REQ0"
+	(global_label "REQ3"
 		(shape input)
 		(at 408.94 132.08 180)

Commit message: Update Input Output Board
Parts:
- added J4: Conn_01x06_Pin, Connector_PinHeader_2.54mm:PinHeader_1x06_P2.54mm_Horizontal, symbol Connector:Conn_01x06_Pin
Connections:
- net LOAD0: now also J4.1 (Pin_1)
- net LOAD1: now also J4.2 (Pin_2)
- net LOAD2: now also J4.3 (Pin_3)
- net LOAD3: now also J4.4 (Pin_4)
- net LOAD4: now also J4.5 (Pin_5)
- net LOAD5: now also J4.6 (Pin_6)
Changed lines of the file:
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@@
 		)
 	)
+	(global_label "LOAD4"
+		(shape input)
+		(at 758.19 308.61 0)
+		(fields_autoplaced yes)
+		(effects
+			(font
+				(size 1.27 1.27)
+			)
+			(justify left)
+		)
+		(property "Intersheetrefs" "${INTERSHEET_REFS}"
+			(at 767.1019 308.61 0)
+			(effects
+				(font
+					(size 1.27 1.27)
+				)
+				(justify left)
+				(hide yes)
+			)
+		)
+	)
 	(global_label "NLOAD4"
 		(shape input)
@@
 		)
 	)
+	(global_label "LOAD5"
+		(shape input)
+		(at 758.19 311.15 0)
+		(fields_autoplaced yes)
+		(effects
+			(font
+				(size 1.27 1.27)
+			)
+			(justify left)
+		)
+		(property "Intersheetrefs" "${INTERSHEET_REFS}"
+			(at 767.1019 311.15 0)
+			(effects
+				(font
+					(size 1.27 1.27)
+				)
+				(justify left)
+				(hide yes)
+			)
+		)
+	)
 	(global_label "REQ3"
 		(shape input)
@@
 		)
 	)
+	(global_label "LOAD1"
+		(shape input)
+		(at 758.19 300.99 0)
+		(fields_autoplaced yes)
+		(effects
+			(font
+				(size 1.27 1.27)
+			)
+			(justify left)
+		)
+		(property "Intersheetrefs" "${INTERSHEET_REFS}"
+			(at 767.1019 300.99 0)
+			(effects
+				(font
+					(size 1.27 1.27)
+				)
+				(justify left)
+				(hide yes)
+			)
+		)
+	)
 	(global_label "INPUT4"
 		(shape input)
@@
 		)
 	)
+	(global_label "LOAD2"
+		(shape input)
+		(at 758.19 303.53 0)
+		(fields_autoplaced yes)
+		(effects
+			(font
+				(size 1.27 1.27)
+			)
+			(justify left)
+		)
+		(property "Intersheetrefs" "${INTERSHEET_REFS}"
+			(at 767.1019 303.53 0)
+			(effects
+				(font
+					(size 1.27 1.27)
+				)
+				(justify left)
+				(hide yes)
+			)
+		)
+	)
 	(global_label "NRESET"
 		(shape input)
@@
 		)
 	)
+	(global_label "LOAD3"
+		(shape input)
+		(at 758.19 306.07 0)
+		(fields_autoplaced yes)
+		(effects
+			(font
+				(size 1.27 1.27)
+			)
+			(justify left)
+		)
+		(property "Intersheetrefs" "${INTERSHEET_REFS}"
+			(at 767.1019 306.07 0)
+			(effects
+				(font
+					(size 1.27 1.27)
+				)
+				(justify left)
+				(hide yes)
+			)
+		)
+	)
 	(global_label "NHALT"
 		(shape input)
@@
 		)
 	)
+	(global_label "LOAD0"
+		(shape input)
+		(at 758.19 298.45 0)
+		(fields_autoplaced yes)
+		(effects
+			(font
+				(size 1.27 1.27)
+			)
+			(justify left)
+		)
+		(property "Intersheetrefs" "${INTERSHEET_REFS}"
+			(at 767.1019 298.45 0)
+			(effects
+				(font
+					(size 1.27 1.27)
+				)
+				(justify left)
+				(hide yes)
+			)
+		)
+	)
 	(global_label "TAP_G5"
 		(shape input)
@@
 					(unit 1)
 				)
+			)
+		)
+	)
+	(symbol
+		(lib_id "Connector:Conn_01x06_Pin")
+		(at 753.11 303.53 0)
+		(unit 1)
+		(exclude_from_sim no)
+		(in_bom yes)
+		(on_board yes)
+		(dnp no)
+		(fields_autoplaced yes)
+		(property "Reference" "J4"
+			(at 753.745 293.37 0)
+			(effects
+				(font
+					(size 1.27 1.27)
+				)
+			)
+		)
+		(property "Value" "Conn_01x06_Pin"
+			(at 753.745 295.91 0)
+			(effects
+				(font
+					(size 1.27 1.27)
+				)
+			)
+		)
+		(property "Footprint" "Connector_PinHeader_2.54mm:PinHeader_1x06_P2.54mm_Horizontal"
+			(at 753.11 303.53 0)
+			(effects
+				(font
+					(size 1.27 1.27)
+				)
+				(hide yes)
+			)
+		)
+		(property "Datasheet" "~"
+			(at 753.11 303.53 0)
+			(effects
+				(font
+					(size 1.27 1.27)
+				)
+				(hide yes)
+			)
+		)
+		(property "Description" "Generic connector, single row, 01x06, script generated"
+			(at 753.11 303.53 0)
+			(effects
+				(font
+					(size 1.27 1.27)
+				)
+				(hide yes)
+			)
+		)
+		(pin "4"
+		)
+		(pin "1"
+		)
+		(pin "2"
+		)
+		(pin "3"
+		)
+		(pin "6"
+		)
+		(pin "5"
+		)
+		(instances
+			(project ""
+				(path "/91c9ff6b-da3f-43a7-8acc-896df24b361f"
+					(reference "J4")
+					(unit 1)
+				)
