File: PCB/Santas Microfactory - Input and Output/Santas Microfactory - Input and Output.kicad_pcb (KiCad board)
At the start: 2 copper layers, 200 x 100 mm, 179 parts, among them J1 Conn_01x04_Pin, J10 Conn_01x14_Pin, J2 Conn_01x08_Pin, J3 Conn_01x10_Pin, J4 Conn_01x10_Pin, J5 Conn_01x10_Pin, J6 Conn_01x10_Pin, J7 Conn_01x06_Pin, J8 Conn_01x10_Pin, J9 Conn_01x10_Pin, SW1 SW_DPDT_x2, SW10 SW_DPDT_x2, SW11 SW_DPDT_x2, SW2 SW_DPDT_x2, SW3 SW_DPDT_x2, SW4 SW_DPDT_x2, SW5 SW_DPDT_x2, SW6 SW_DPDT_x2, SW7 SW_DPDT_x2, SW8 SW_DPDT_x2, SW9 SW_DPDT_x2

Commit message: Input Output Board Finished
Parts:
- J1, J10, J2, J3, J4, J5, J6, J7, J8, J9: moved to B.Cu
- moved J1 268.5 mm to (239.0, 84.8)
- moved J5 249.6 mm to (225.2, 114.2)
- moved J6 241.1 mm to (221.2, 114.2)
- moved J2 241.1 mm to (239.0, 54.7), turned to 180 degrees
- moved J3 187.0 mm to (149.9, 122.1), turned to -90 degrees
- moved J4 181.5 mm to (149.9, 118.0), turned to -90 degrees
- moved J7 169.5 mm to (155.0, 143.2), turned to -90 degrees
- moved J10 130.7 mm to (85.8, 121.0), turned to -90 degrees
- moved J9 83.8 mm to (76.5, 81.2)
- moved J8 78.2 mm to (66.2, 81.2)
- moved D59 23.0 mm to (202.0, 69.5)
- moved R59 23.0 mm to (202.0, 64.2)
Connections:
- J8 pad 10: TAP_C9 -> OUT_C9
- J8 pad 3: TAP_C2 -> OUT_C2
- J8 pad 4: TAP_C3 -> OUT_C3
- J8 pad 6: TAP_C5 -> OUT_C5
- J8 pad 7: TAP_C6 -> OUT_C6
- J8 pad 9: TAP_C8 -> OUT_C8
- J9 pad 10: TAP_G9 -> OUT_G9
- J9 pad 3: TAP_G2 -> OUT_G2
- J9 pad 4: TAP_G3 -> OUT_G3
- J9 pad 6: TAP_G5 -> OUT_G5
- J9 pad 7: TAP_G6 -> OUT_G6
- J9 pad 9: TAP_G8 -> OUT_G8
Routing:
- net CLK: track 0.00 -> 211.0 mm
- net HALT: track 0.00 -> 202.6 mm
- net OUT_C9: track 0.00 -> 134.8 mm
- net OUT_C8: track 0.00 -> 125.0 mm
- net OUT_G9: track 0.00 -> 121.5 mm
- net RESET: track 7.74 -> 128.5 mm
- net OUT_C7: track 0.00 -> 115.2 mm
- net OUT_G8: track 0.00 -> 111.7 mm
- net OUT_C6: track 0.00 -> 105.5 mm
- net OUT_G7: track 0.00 -> 102.0 mm
- net INPUT5: track 0.00 -> 97.8 mm
- net OUT_C5: track 0.00 -> 95.7 mm
- net OUT_G6: track 0.00 -> 92.2 mm
- net OUT_C4: track 0.00 -> 85.9 mm
- net INPUT4: track 0.00 -> 85.7 mm
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- added copper zone on B.Cu, net GND
- added copper zone on F.Cu, net GND

Commit message: All silkscreen additions + Gerbers and CAD files
Silkscreen and Gerbers are done, but I plan on using the CAD to create additional renders.
Parts:
- added G***: LOGO, LOGO, F.Cu at (83.6, 94.8)
- added G***: LOGO, LOGO, B.Cu at (217.2, 129.2)
- added G***: LOGO, LOGO, B.Cu at (87.6, 95.7)
- added G***: LOGO, LOGO, B.Cu at (245.0, 117.0)
Other:
- board text added: "@->-->---"
- board text added: "An entirely Diode Transistor Logic {dblquote}Computer{dblquote} Game!"
- board text added: "C0,1,2"
- board text added: "C5,4,3"
- board text added: "CHUTE0"
- board text added: "CHUTE1"
- board text added: "CHUTE2"
- board text added: "CHUTE3"
- board text added: "CHUTE4"
- board text added: "CHUTE5"
- board text added: "CLOCK"
- board text added: "COAL CONVEYOR"
- board text added: "Designed by Logan Peterson"
- board text added: "G0,1,2"
- board text added: "G5,4,3"
- board text added: "GIFT CONVEYOR"
- board text added: "HALT"
- board text added: "HEALTH"
- board text added: "INPUT"
- board text added: "Input and Output"
- board text added: "RESET"
- board text added: "Randomize the outputs:"
- board text added: "SCORE"
- board text added: "SEED1"
- board text added: "SEED2"
- board text added: "SEED3"
- board text added: "SEED4"
- board text added: "SYSTEM"
- board text added: "Santas Microfactory"
- board text added: "{dblquote}Making sand think{dblquote}"
