File: PCB/Santas Microfactory - Chutes PCB 1/Santas Microfactory - Chutes PCB 1.kicad_pcb (KiCad board)
At the start: 4 copper layers, 200 x 191.1 mm, 39 parts, among them J1 Conn_01x10_Pin, J2 Conn_01x10_Pin, J4 Bus_PCI_Express_x16

Commit message: All silkscreen additions + Gerbers and CAD files
Silkscreen and Gerbers are done, but I plan on using the CAD to create additional renders.
Parts:
- added G***: LOGO, LOGO, F.Cu at (60.8, 123.8)
- added G***: LOGO, LOGO, F.Cu at (63.0, 177.5)
- added G***: LOGO, LOGO, F.Cu at (56.5, 63.2)
- added G***: LOGO, LOGO, B.Cu at (56.2, 130.0)
Other:
- board text added: "C0,1,2"
- board text added: "CHUTES PCB 1"
- board text added: "Designed by Logan Peterson"
- board text added: "G0,1,2"
