File: PCB/Santas Microfactory - Chutes PCB 2/Santas Microfactory - Chutes PCB 2.kicad_pcb (KiCad board)
At the start: 4 copper layers, 200 x 191.1 mm, 39 parts, among them J1 Conn_01x10_Pin, J2 Conn_01x10_Pin, J4 Bus_PCI_Express_x16

Commit message: All silkscreen additions + Gerbers and CAD files
Silkscreen and Gerbers are done, but I plan on using the CAD to create additional renders.
Parts:
- added G***: LOGO, LOGO, F.Cu at (60.0, 69.0)
- added G***: LOGO, LOGO, F.Cu at (60.0, 152.2)
- added G***: LOGO, LOGO, B.Cu at (59.5, 122.5)
Other:
- board text added: "C5,4,3"
- board text added: "CHUTES PCB 2"
- board text added: "Designed by Logan Peterson"
- board text added: "G5,4,3"
