File: PCB/Santas Microfactory - Scoring and Health/Santas Microfactory - Scoring and Health.kicad_pcb (KiCad board)
At the start: 2 copper layers, 200 x 191.1 mm, 630 parts, among them J2 Conn_01x08_Pin, J3 Conn_01x04_Pin, J4 Bus_PCI_Express_x16, Q1 NPN, Q10 NPN, Q11 NPN, Q12 NPN, Q13 NPN, Q14 NPN, Q15 NPN, Q16 NPN, Q17 NPN, Q18 NPN, Q19 NPN, Q2 NPN, Q20 NPN, Q21 NPN, Q22 NPN, Q23 NPN, Q24 NPN, Q25 NPN, Q26 NPN, Q27 NPN, Q28 NPN, Q29 NPN, Q3 NPN, Q30 NPN, Q31 NPN, Q32 NPN, Q33 NPN, Q34 NPN, Q35 NPN, Q36 NPN, Q37 NPN, Q38 NPN, Q39 NPN, Q4 NPN, Q40 NPN, Q41 NPN, Q42 NPN, Q43 NPN, Q44 NPN, Q45 NPN, Q46 NPN, Q47 NPN, Q48 NPN, Q49 NPN, Q5 NPN, Q50 NPN, Q51 NPN, Q52 NPN, Q53 NPN, Q54 NPN, Q55 NPN, Q56 NPN, Q57 NPN, Q58 NPN, Q59 NPN, Q6 NPN, Q60 NPN, Q61 NPN, Q62 NPN, Q63 NPN, Q64 NPN, Q65 NPN, Q66 NPN, Q67 NPN, Q68 NPN, Q69 NPN, Q7 NPN, Q70 NPN, Q71 NPN, Q72 NPN, Q73 NPN, Q74 NPN, Q75 NPN, Q76 NPN, Q77 NPN, Q78 NPN, Q79 NPN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

Commit message: All silkscreen additions + Gerbers and CAD files
Silkscreen and Gerbers are done, but I plan on using the CAD to create additional renders.
Parts:
- added G***: LOGO, LOGO, F.Cu at (51.8, 161.0)
- added G***: LOGO, LOGO, F.Cu at (192.1, 42.6)
- added G***: LOGO, LOGO, F.Cu at (75.4, 44.9)
- added G***: LOGO, LOGO, F.Cu at (219.8, 172.8)
Other:
- board text added: "Designed by: Logan Peterson"
- board text added: "HEALTH"
- board text added: "SCORE"
- board text added: "Scoring and Health"
